File: circuits/base_circuit/base_circuit.brd (EAGLE design)
At the start: 53 x 85.1 mm, 33 parts, among them U1 ARDUINO-MEGAFULL

Commit message: changed the whole circuit to use speed control for individula motors and also added connections for top plate design leds
Parts:
- removed D1, D2, D3, D4: (no value), diode4:DIODE-1N4148
- removed R1, R2, R3, R4: 4.7k, rcl:0207/12
- moved CN1 240.0 mm to (40.6, 73.0), turned to 90 degrees
- moved D5 210.8 mm to (22.9, 54.0)
- moved J1 201.3 mm to (10.2, 54.0)
- moved R12 163.1 mm to (38.1, 39.4), turned to 180 degrees
- moved CN2 161.3 mm to (10.2, 24.8), turned to 90 degrees
- moved R11 152.6 mm to (38.1, 33.0), turned to 180 degrees
- moved R10 142.0 mm to (38.1, 26.7), turned to 180 degrees
- moved R9 131.5 mm to (38.1, 20.3), turned to 180 degrees
- moved R8 121.1 mm to (38.1, 14.0), turned to 180 degrees
- moved R7 110.7 mm to (38.1, 7.62), turned to 180 degrees
- moved QN6 109.2 mm to (26.0, 36.8), turned to 180 degrees
- moved QN5 94.9 mm to (26.0, 30.5), turned to 180 degrees
- moved MOTOR1 84.7 mm to (94.0, 65.4)
- moved QN4 80.7 mm to (26.0, 24.1), turned to 180 degrees
- moved QN3 66.7 mm to (26.0, 17.8), turned to 180 degrees
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Connections:
- removed net BRAKEPIN: MOTOR1.1, MOTOR2.1, MOTOR3.1, MOTOR4.1, U1.14
- removed net N$1: D1.C, MOTOR1.4
- removed net N$2: D2.C, MOTOR2.4
- removed net N$25: CN1.4
- removed net N$26: CN1.3
- removed net N$3: D3.C, MOTOR3.4
- removed net N$33: CN1.2
- removed net N$34: CN1.1
- removed net N$4: D4.C, MOTOR4.4
- removed net SPEEDPIN: MOTOR1.6, MOTOR2.6, MOTOR3.6, MOTOR4.6, U1.46
- removed net TACHO-M1: D1.A, R1.1, U1.2
- removed net TACHO-M2: D2.A, R2.1, U1.3
- removed net TACHO-M3: D3.A, R3.1, U1.4
- removed net TACHO-M4: D4.A, R4.1, U1.5
- new net BRAKE-M1: MOTOR1.1, U1.52
- new net BRAKE-M2: MOTOR2.1, U1.44
- new net BRAKE-M3: MOTOR3.1, U1.36
- new net BRAKE-M4: MOTOR4.1, U1.28
- new net FEEDBACK_IN1: CN1.3, U1.22
- new net FEEDBACK_IN2: CN1.4, U1.23
- new net FEEDBACK_INT1: CN1.1, U1.18
- new net FEEDBACK_INT2: CN1.2, U1.19
- new net SPEED-M1: MOTOR1.6, U1.46
- new net SPEED-M2: MOTOR2.6, U1.4
- new net SPEED-M3: MOTOR3.6, U1.3
- new net SPEED-M4: MOTOR4.6, U1.2
- net DIR-M1: now also U1.48; no longer U1.16
- net DIR-M2: now also U1.40; no longer U1.36
- net DIR-M3: now also U1.32; no longer U1.40
- net DIR-M4: now also U1.24; no longer U1.44
- net DIS-M1: now also U1.50; no longer U1.17
- net DIS-M2: now also U1.42; no longer U1.34
- net DIS-M3: now also U1.34; no longer U1.38
- net DIS-M4: now also U1.26; no longer U1.42
- net GND: now also U1.GND@2, U1.GND@3; no longer U1.GND@0, U1.GND@1
- net L1: now also U1.12
- net L2: now also U1.11
- net L3: now also U1.10
- net L4: now also U1.9
- net L5: now also U1.8
- net L6: now also U1.7
- net VCC: no longer R1.2, R2.2, R3.2, R4.2
Routing:
- net VCC/2: track 0.00 -> 180.6 mm
- net BRAKEPIN: track 76.2 -> 0.00 mm
- net SPEEDPIN: track 75.0 -> 0.00 mm
- net SPEED-M2: track 0.00 -> 45.3 mm
- net VCC: track 90.8 -> 49.9 mm
- net TACHO-M4: track 40.5 -> 0.00 mm
- net SPEED-M3: track 0.00 -> 34.1 mm
- net TACHO-M3: track 29.9 -> 0.00 mm
- net SPEED-M4: track 0.00 -> 25.5 mm
- net SPEED-M1: track 0.00 -> 20.4 mm
- net TACHO-M2: track 19.4 -> 0.00 mm
- net N$32: track 0.00 -> 17.3 mm
- net N$27: track 0.00 -> 17.3 mm
- net DIS-M4: track 25.1 -> 8.15 mm
- net L6: track 0.00 -> 16.5 mm
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Other:
- board size 53 x 85.1 mm -> 104.4 x 85.7 mm

Commit message: edited BRD file
Parts:
- moved J1 19.9 mm to (20.3, 71.1), turned to 270 degrees
- moved IMU 6.35 mm to (59.7, 9.53)
- moved MOTOR1 6.35 mm to (87.6, 65.4)
- moved R5 6.35 mm to (57.8, 19.1)
- moved CN1 6.35 mm to (34.3, 73.0)
- moved JP1 6.35 mm to (47.0, 2.54)
- moved MOTOR4 6.35 mm to (57.1, 65.4)
- moved QN1 6.35 mm to (19.7, 5.08)
- moved QN2 6.35 mm to (19.7, 11.4)
- moved QN3 6.35 mm to (19.7, 17.8)
- moved QN4 6.35 mm to (19.7, 24.1)
- moved QN5 6.35 mm to (19.7, 30.5)
- moved QN6 6.35 mm to (19.7, 36.8)
- moved R10 6.35 mm to (31.8, 26.7)
- moved R11 6.35 mm to (31.8, 33.0)
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Routing:
- net GND: track 87.9 -> 216.2 mm
- net FEEDBACK_IN2: track 0.00 -> 19.7 mm
- net FEEDBACK_IN1: track 0.00 -> 17.2 mm
- net FEEDBACK_INT2: track 0.00 -> 15.3 mm
- net FEEDBACK_INT1: track 0.00 -> 15.3 mm
- net N$24: track 0.00 -> 6.68 mm
- net VCC/2: track 180.6 -> 185.0 mm
Other:
- board size 104.4 x 85.7 mm -> 98.7 x 85.1 mm
- board text added: "Mk III"
- board text added: "v10"
- board text removed: "Mk II"
- board text removed: "v6"
