Commit message: updates to RPlidar

File: src/lidar_robot/xacro/base.xacro (robot description, xacro)
@@ -1,53 +1,54 @@
 <?xml version="1.0"?>
 <robot xmlns:xacro="http://www.ros.org/wiki/xacro" name="lidar_robot">
+    <xacro:property name="pi" value="3.14159265359"/>
     <link name="base_link">
         <inertial>
-            <origin xyz="-0.0099877 -7.87679999999704E-06 0.048337" rpy="0 0 0" />
-            <mass value="6.0202" />
-            <inertia ixx="0.193404669051707" ixy="-1.57451867364915E-06" ixz="7.52537384896092E-06" iyy="1.01182032486468E-06" iyz="-0.193412304186565" izz="-1.01182032483072E-06" />
+            <origin xyz="-0.0099877 -7.87679999999704E-06 0.048337" rpy="0 0 0"/>
+            <mass value="6.0202"/>
+            <inertia ixx="0.193404669051707" ixy="-1.57451867364915E-06" ixz="7.52537384896092E-06" iyy="1.01182032486468E-06" iyz="-0.193412304186565" izz="-1.01182032483072E-06"/>
         </inertial>
         <visual>
-            <origin xyz="0 0 0" rpy="1.5707963267949 0 0" />
+            <origin xyz="0 0 0" rpy="${pi/2} 0 0"/>
             <geometry>
-                <mesh filename="package://lidar_robot/meshes/base.stl" />
+                <mesh filename="package://lidar_robot/meshes/base.stl"/>
             </geometry>
             <material name="">
-                <color rgba="0.8 0.8 0.8 1" />
+                <color rgba="0.8 0.8 0.8 1"/>
             </material>
         </visual>
         <collision>
-            <origin xyz="0 0 0" rpy="${pi/2} 0 0" />
+            <origin xyz="0 0 0" rpy="${pi/2} 0 0"/>
             <geometry>
-                <mesh filename="package://lidar_robot/meshes/base.stl" />
+                <mesh filename="package://lidar_robot/meshes/base.stl"/>
             </geometry>
         </collision>
     </link>
-  <link name="rplidar">
-    <collision>
-      <origin xyz="0 0 0" rpy="0 0 0"/>
-      <geometry>
-    <box size="0.1 0.1 0.1"/>
-      </geometry>
-    </collision>
-    <visual>
-      <origin xyz="0 0 0" rpy="0 0 0"/>
-      <geometry>
-        <mesh filename="package://lidar_robot/meshes/rplidar.stl"/>
-      </geometry>
-      <material name="">
-                <color rgba="0.1 0.1 0.1 1" />
-      </material>
-    </visual>
-    <inertial>
-      <origin xyz="0.010606 0.000652570000000001 0.015976" rpy="0 0 0" />
-      <mass value="0.095964" />
-      <inertia ixx="4.20678723401718E-05" ixy="-1.30097836316357E-05" ixz="4.33129403884459E-07" iyy="1.48659304158389E-06" iyz="-7.76207439662319E-05" izz="-1.48659304158388E-06" />
-    </inertial>
-  </link>
-  <joint name="rplidar_joint" type="fixed">
-    <axis xyz="0 1 0" />
-    <origin xyz="0 0 0" rpy="0 0 0"/>
-    <child link="rplidar"/>
-    <parent link="base_link"/>
-  </joint>
+    <link name="rplidar">
+        <collision>
+            <origin xyz="0 0 0" rpy="0 0 0"/>
+            <geometry>
+                <box size="0.1 0.1 0.1"/>
+            </geometry>
+        </collision>
+        <visual>
+            <origin xyz="0 0 0.11675" rpy="${pi/2} 0 0"/>
+            <geometry>
+                <mesh filename="package://lidar_robot/meshes/rplidar.stl"/>
+            </geometry>
+            <material name="">
+                <color rgba="0.1 0.1 0.1 1"/>
+            </material>
+        </visual>
+        <inertial>
+            <origin xyz="0.010606 0.000652570000000001 0.015976" rpy="0 0 0"/>
+            <mass value="0.095964"/>
+            <inertia ixx="4.20678723401718E-05" ixy="-1.30097836316357E-05" ixz="4.33129403884459E-07" iyy="1.48659304158389E-06" iyz="-7.76207439662319E-05" izz="-1.48659304158388E-06"/>
+        </inertial>
+    </link>
+    <joint name="rplidar_joint" type="fixed">
+        <axis xyz="1 0 0"/>
+        <origin xyz="0 2 0" rpy="0 0 0"/>
+        <child link="rplidar"/>
+        <parent link="base_link"/>
+    </joint>
 </robot>
