Commit message: Updated RVIZ
Files working with tf jointstatepublisher and robot_tf_publisher perfectly on rviz as well as website

File: src/lidar_robot/xacro/rviz.xacro (robot description, xacro)
@@ -80,5 +80,5 @@
     <link name="shaft_1">
         <visual>
-            <origin xyz="${-(c_clamp_dist+0.01)} 0 0.045" rpy="0 0 ${pi}"/>
+            <origin xyz="0 0 0" rpy="0 0 0"/>
             <geometry>
                 <mesh filename="package://lidar_robot/models/motor_shaft.stl" scale="0.001 0.001 0.001"/>
@@ -87,11 +87,13 @@
         </visual>
     </link>
-    <joint name="motor_shaft_1" type="fixed">
+    <joint name="motor_shaft_1" type="continuous">
         <parent link="motor_1"/>
         <child link="shaft_1"/>
+        <axis xyz="1 0 0"/>
+        <origin xyz="${-(c_clamp_dist+0.01)} 0 0.045" rpy="0 0 ${pi}"/>
     </joint>
     <link name="wheel_1">
         <visual>
-            <origin xyz="-${(c_clamp_dist+0.03)} 0 0.045" rpy="0 0 ${-pi/2}"/>
+            <origin xyz="0.02 0 0" rpy="0 0 ${pi/2}"/>
             <geometry>
                 <mesh filename="package://lidar_robot/models/wheel2.dae"/>
@@ -132,5 +134,5 @@
     <link name="shaft_2">
         <visual>
-            <origin xyz="0 ${(c_clamp_dist+0.01)} 0.045" rpy="0 0 ${pi/2}"/>
+            <origin xyz="0 0 0" rpy="0 0 0"/>
             <geometry>
                 <mesh filename="package://lidar_robot/models/motor_shaft.stl" scale="0.001 0.001 0.001"/>
@@ -139,11 +141,12 @@
         </visual>
     </link>
-    <joint name="motor_shaft_2" type="fixed">
+    <joint name="motor_shaft_2" type="continuous">
         <parent link="motor_2"/>
         <child link="shaft_2"/>
+        <origin xyz="0 ${(c_clamp_dist+0.01)} 0.045" rpy="0 0 ${pi/2}"/>
     </joint>
     <link name="wheel_2">
         <visual>
-            <origin xyz="0 ${(c_clamp_dist+0.03)} 0.045" rpy="0 0 ${pi}"/>
+            <origin xyz="0.02 0 0" rpy="0 0 ${pi/2}"/>
             <geometry>
                 <mesh filename="package://lidar_robot/models/wheel2.dae"/>
@@ -184,5 +187,5 @@
     <link name="shaft_3">
         <visual>
-            <origin xyz="${(c_clamp_dist+0.01)} 0 0.045" rpy="0 0 0"/>
+            <origin xyz="0 0 0" rpy="0 0 0"/>
             <geometry>
                 <mesh filename="package://lidar_robot/models/motor_shaft.stl" scale="0.001 0.001 0.001"/>
@@ -191,11 +194,12 @@
         </visual>
     </link>
-    <joint name="motor_shaft_3" type="fixed">
+    <joint name="motor_shaft_3" type="continuous">
         <parent link="motor_3"/>
         <child link="shaft_3"/>
+        <origin xyz="${(c_clamp_dist+0.01)} 0 0.045" rpy="0 0 0"/>
     </joint>
     <link name="wheel_3">
         <visual>
-            <origin xyz="${(c_clamp_dist+0.03)} 0 0.045" rpy="0 0 ${pi/2}"/>
+            <origin xyz="0.02 0 0" rpy="0 0 ${pi/2}"/>
             <geometry>
                 <mesh filename="package://lidar_robot/models/wheel2.dae"/>
@@ -236,5 +240,5 @@
     <link name="shaft_4">
         <visual>
-            <origin xyz="0 ${-(c_clamp_dist+0.01)} 0.045" rpy="0 0 ${-pi/2}"/>
+            <origin xyz="0 0 0" rpy="0 0 0"/>
             <geometry>
                 <mesh filename="package://lidar_robot/models/motor_shaft.stl" scale="0.001 0.001 0.001"/>
@@ -243,11 +247,12 @@
         </visual>
     </link>
-    <joint name="motor_shaft_4" type="fixed">
+    <joint name="motor_shaft_4" type="continuous">
         <parent link="motor_4"/>
         <child link="shaft_4"/>
+        <origin xyz="0 ${-(c_clamp_dist+0.01)} 0.045" rpy="0 0 ${-pi/2}"/>
     </joint>
     <link name="wheel_4">
         <visual>
-            <origin xyz="0 ${-(c_clamp_dist+0.03)} 0.045" rpy="0 0 0"/>
+            <origin xyz="0.02 0 0" rpy="0 0 ${pi/2}"/>
             <geometry>
                 <mesh filename="package://lidar_robot/models/wheel2.dae"/>
