Commit message: Added circuit plate

File: src/lidar_robot/xacro/robot.xacro (robot description, xacro)
@@ -15,5 +15,5 @@
     <link name="base_link">
         <visual>
-            <origin xyz="0 0 0" rpy="${pi/2} 0 0"/>
+            <origin xyz="0.01 0 0" rpy="${pi/2} 0 0"/>
             <geometry>
                 <mesh filename="package://lidar_robot/models/base.stl" scale="0.001 0.001 0.001"/>
@@ -22,5 +22,5 @@
         </visual>
     </link>
-    <!-- =======================================================Wheel 4====================================================================== -->
+    <!-- =======================================================Wheel 1====================================================================== -->
     <link name="c_clamp_1">
         <visual>
@@ -245,9 +245,11 @@
     <link name="top_plate">
         <visual>
-            <origin xyz="0 0 0.0836" rpy="${pi/2} 0 0"/>
+            <origin xyz="0.01 0 0.0836" rpy="${pi/2} 0 0"/>
             <geometry>
                 <mesh filename="package://lidar_robot/models/top_plate.stl" scale="0.001 0.001 0.001"/>
             </geometry>
-            <material name="plastic"/>
+            <material name="blue">
+                <color rgba="0 0 1.0 1"/>
+            </material>
         </visual>
     </link>
@@ -256,3 +258,17 @@
         <child link="top_plate"/>
     </joint>
+    <!-- ======================================================= Circuit Plate ====================================================================== -->
+    <link name="circuit_plate">
+        <visual>
+            <origin xyz="0 0 0.093" rpy="${pi/2} 0 ${pi/4}"/>
+            <geometry>
+                <mesh filename="package://lidar_robot/models/circuit_plate.stl" scale="0.001 0.001 0.001"/>
+            </geometry>
+            <material name="plastic"/>
+        </visual>
+    </link>
+    <joint name="base_link_circuit_plate" type="fixed">
+        <parent link="top_plate"/>
+        <child link="circuit_plate"/>
+    </joint>
 </robot>

Commit message: Updated server.js for spawn, printing stdout and stderr now

File: src/lidar_robot/xacro/robot.xacro (robot description, xacro)
@@ -13,4 +13,9 @@
         <color rgba="0.95 0.95 0.95 1"/>
     </material>
+    <material name="blue">
+        <color rgba="0 0 1.0 1"/>
+    </material>
+    <xacro:property name="c_clamp_dist" value="2.1"/>
+    <xacro:property name="the_radius" value="2.1"/>
     <link name="base_link">
         <visual>
@@ -249,7 +254,5 @@
                 <mesh filename="package://lidar_robot/models/top_plate.stl" scale="0.001 0.001 0.001"/>
             </geometry>
-            <material name="blue">
-                <color rgba="0 0 1.0 1"/>
-            </material>
+            <material name="blue"/>
         </visual>
     </link>

Commit message: Changed distance from center Changed distance from center of c clamp motor shaft and wheel to a variable

File: src/lidar_robot/xacro/robot.xacro (robot description, xacro)
@@ -16,6 +16,5 @@
         <color rgba="0 0 1.0 1"/>
     </material>
-    <xacro:property name="c_clamp_dist" value="2.1"/>
-    <xacro:property name="the_radius" value="2.1"/>
+    <xacro:property name="c_clamp_dist" value="0.31"/>
     <link name="base_link">
         <visual>
@@ -30,5 +29,5 @@
     <link name="c_clamp_1">
         <visual>
-            <origin xyz="-0.32 0.05 0.09" rpy="${pi/2} 0 0"/>
+            <origin xyz="${-c_clamp_dist} 0.05 0.09" rpy="${pi/2} 0 0"/>
             <geometry>
                 <mesh filename="package://lidar_robot/models/c_clamp.stl" scale="0.001 0.001 0.001"/>
@@ -43,5 +42,5 @@
     <link name="motor_1">
         <visual>
-            <origin xyz="-0.308 0 0.045" rpy="${pi/2} 0 ${pi/2}"/>
+            <origin xyz="${-(c_clamp_dist-0.012)} 0 0.045" rpy="${pi/2} 0 ${pi/2}"/>
             <geometry>
                 <mesh filename="package://lidar_robot/models/motor.stl" scale="0.001 0.001 0.001"/>
@@ -56,5 +55,5 @@
     <link name="shaft_1">
         <visual>
-            <origin xyz="-0.33 0 0.045" rpy="0 0 ${pi}"/>
+            <origin xyz="${-(c_clamp_dist+0.01)} 0 0.045" rpy="0 0 ${pi}"/>
             <geometry>
                 <mesh filename="package://lidar_robot/models/motor_shaft.stl" scale="0.001 0.001 0.001"/>
@@ -69,5 +68,5 @@
     <link name="wheel_1">
         <visual>
-            <origin xyz="-0.365 0 0.045" rpy="0 0 ${pi/2}"/>
+            <origin xyz="${-(c_clamp_dist+0.03)} 0 0.045" rpy="0 0 ${pi/2}"/>
             <geometry>
                 <mesh filename="package://lidar_robot/models/wheel2.dae"/>
@@ -85,5 +84,5 @@
     <link name="c_clamp_2">
         <visual>
-            <origin xyz="0.05 0.32 0.09" rpy="${pi/2} 0 -${pi/2}"/>
+            <origin xyz="0.05 ${c_clamp_dist} 0.09" rpy="${pi/2} 0 -${pi/2}"/>
             <geometry>
                 <mesh filename="package://lidar_robot/models/c_clamp.stl" scale="0.001 0.001 0.001"/>
@@ -98,5 +97,5 @@
     <link name="motor_2">
         <visual>
-            <origin xyz="0 0.308 0.045" rpy="${pi/2} -${pi} 0"/>
+            <origin xyz="0 ${(c_clamp_dist-0.012)} 0.045" rpy="${pi/2} -${pi} 0"/>
             <geometry>
                 <mesh filename="package://lidar_robot/models/motor.stl" scale="0.001 0.001 0.001"/>
@@ -111,5 +110,5 @@
     <link name="shaft_2">
         <visual>
-            <origin xyz="0 0.33 0.045" rpy="0 0 ${pi/2}"/>
+            <origin xyz="0 ${(c_clamp_dist+0.01)} 0.045" rpy="0 0 ${pi/2}"/>
             <geometry>
                 <mesh filename="package://lidar_robot/models/motor_shaft.stl" scale="0.001 0.001 0.001"/>
@@ -124,5 +123,5 @@
     <link name="wheel_2">
         <visual>
-            <origin xyz="0 0.35 0.045" rpy="0 0 ${pi}"/>
+            <origin xyz="0 ${(c_clamp_dist+0.03)} 0.045" rpy="0 0 ${pi}"/>
             <geometry>
                 <mesh filename="package://lidar_robot/models/wheel2.dae"/>
@@ -140,5 +139,5 @@
     <link name="c_clamp_3">
         <visual>
-            <origin xyz="0.32 -0.05 0.09" rpy="${pi/2} 0 ${pi}"/>
+            <origin xyz="${c_clamp_dist} -0.05 0.09" rpy="${pi/2} 0 ${pi}"/>
             <geometry>
                 <mesh filename="package://lidar_robot/models/c_clamp.stl" scale="0.001 0.001 0.001"/>
@@ -153,5 +152,5 @@
     <link name="motor_3">
         <visual>
-            <origin xyz="0.308 0 0.045" rpy="${pi/2} 0 -${pi/2}"/>
+            <origin xyz="${(c_clamp_dist-0.012)} 0 0.045" rpy="${pi/2} 0 -${pi/2}"/>
             <geometry>
                 <mesh filename="package://lidar_robot/models/motor.stl" scale="0.001 0.001 0.001"/>
@@ -166,5 +165,5 @@
     <link name="shaft_3">
         <visual>
-            <origin xyz="0.33 0 0.045" rpy="0 0 0"/>
+            <origin xyz="${(c_clamp_dist+0.01)} 0 0.045" rpy="0 0 0"/>
             <geometry>
                 <mesh filename="package://lidar_robot/models/motor_shaft.stl" scale="0.001 0.001 0.001"/>
@@ -179,5 +178,5 @@
     <link name="wheel_3">
         <visual>
-            <origin xyz="0.35 0 0.045" rpy="0 0 ${pi/2}"/>
+            <origin xyz="${(c_clamp_dist+0.03)} 0 0.045" rpy="0 0 ${pi/2}"/>
             <geometry>
                 <mesh filename="package://lidar_robot/models/wheel2.dae"/>
@@ -195,5 +194,5 @@
     <link name="c_clamp_4">
         <visual>
-            <origin xyz="-0.05 -0.32 0.09" rpy="${pi/2} 0 ${pi/2}"/>
+            <origin xyz="-0.05 ${-c_clamp_dist} 0.09" rpy="${pi/2} 0 ${pi/2}"/>
             <geometry>
                 <mesh filename="package://lidar_robot/models/c_clamp.stl" scale="0.001 0.001 0.001"/>
@@ -208,5 +207,5 @@
     <link name="motor_4">
         <visual>
-            <origin xyz="0 -0.308 0.045" rpy="${pi/2} 0 ${pi}"/>
+            <origin xyz="0 ${-(c_clamp_dist-0.012)} 0.045" rpy="${pi/2} 0 ${pi}"/>
             <geometry>
                 <mesh filename="package://lidar_robot/models/motor.stl" scale="0.001 0.001 0.001"/>
@@ -221,5 +220,5 @@
     <link name="shaft_4">
         <visual>
-            <origin xyz="0 -0.33 0.045" rpy="0 0 ${-pi/2}"/>
+            <origin xyz="0 ${-(c_clamp_dist+0.01)} 0.045" rpy="0 0 ${-pi/2}"/>
             <geometry>
                 <mesh filename="package://lidar_robot/models/motor_shaft.stl" scale="0.001 0.001 0.001"/>
@@ -234,5 +233,5 @@
     <link name="wheel_4">
         <visual>
-            <origin xyz="0 -0.35 0.045" rpy="0 0 0"/>
+            <origin xyz="0 ${-(c_clamp_dist+0.03)} 0.045" rpy="0 0 0"/>
             <geometry>
                 <mesh filename="package://lidar_robot/models/wheel2.dae"/>

Commit message: Added Feedback and Studs for it

File: src/lidar_robot/xacro/robot.xacro (robot description, xacro)
@@ -16,4 +16,7 @@
         <color rgba="0 0 1.0 1"/>
     </material>
+    <material name="bronze">
+        <color rgba="0.8039 0.498 0.196 1"/>
+    </material>
     <xacro:property name="c_clamp_dist" value="0.31"/>
     <link name="base_link">
@@ -274,3 +277,40 @@
         <child link="circuit_plate"/>
     </joint>
+    <!-- ======================================================= feedback ====================================================================== -->
+    <link name="feedback">
+        <visual>
+            <origin xyz="0.063 0.1 -0.06" rpy="${pi/2} 0 ${pi/4}"/>
+            <geometry>
+                <mesh filename="package://lidar_robot/models/feedback.stl" scale="0.001 0.001 0.001"/>
+            </geometry>
+            <material name="aluminium_dark"/>
+        </visual>
+    </link>
+    <joint name="base_link_feedback" type="fixed">
+        <parent link="base_link"/>
+        <child link="feedback"/>
+    </joint>
+    <xacro:macro name="stud" params="myname x y z parent">
+        <link name="${myname}">
+            <visual>
+                <origin xyz="${x} ${y} ${z}" rpy="${pi/2} 0 0"/>
+                <geometry>
+                    <mesh filename="package://lidar_robot/models/stud.stl" scale="0.001 0.001 0.001"/>
+                </geometry>
+                <material name="bronze"/>
+            </visual>
+        </link>
+        <joint name="${parent}_${myname}" type="fixed">
+            <parent link="${parent}"/>
+            <child link="${myname}"/>
+        </joint>
+    </xacro:macro>
+    <xacro:stud myname="s1" x="0.073" y="0.06" z="0.006" parent="feedback"/>
+    <xacro:stud myname="s2" x="-0.073" y="0.06" z="0.006" parent="feedback"/>
+    <xacro:stud myname="s3" x="0.073" y="-0.06" z="0.006" parent="feedback"/>
+    <xacro:stud myname="s4" x="-0.073" y="-0.06" z="0.006" parent="feedback"/>
+    <xacro:stud myname="s5" x="0.06" y="0.0735" z="0.006" parent="feedback"/>
+    <xacro:stud myname="s6" x="-0.06" y="0.0735" z="0.006" parent="feedback"/>
+    <xacro:stud myname="s7" x="0.06" y="-0.0735" z="0.006" parent="feedback"/>
+    <xacro:stud myname="s8" x="-0.06" y="-0.0735" z="0.006" parent="feedback"/>
 </robot>
