Commit message: Added RPlidar base in model

File: src/lidar_robot/xacro/robot.xacro (robot description, xacro)
@@ -20,275 +20,4 @@
     </material>
     <xacro:property name="c_clamp_dist" value="0.31"/>
-    <link name="base_link">
-        <visual>
-            <origin xyz="0.01 0 0" rpy="${pi/2} 0 0"/>
-            <geometry>
-                <mesh filename="package://lidar_robot/models/base.stl" scale="0.001 0.001 0.001"/>
-            </geometry>
-            <material name="transparent_acrylic"/>
-        </visual>
-    </link>
-    <!-- =======================================================Wheel 1====================================================================== -->
-    <link name="c_clamp_1">
-        <visual>
-            <origin xyz="${-c_clamp_dist} 0.05 0.09" rpy="${pi/2} 0 0"/>
-            <geometry>
-                <mesh filename="package://lidar_robot/models/c_clamp.stl" scale="0.001 0.001 0.001"/>
-            </geometry>
-            <material name="aluminium"/>
-        </visual>
-    </link>
-    <joint name="base_c_clamp_1" type="fixed">
-        <parent link="base_link"/>
-        <child link="c_clamp_1"/>
-    </joint>
-    <link name="motor_1">
-        <visual>
-            <origin xyz="${-(c_clamp_dist-0.012)} 0 0.045" rpy="${pi/2} 0 ${pi/2}"/>
-            <geometry>
-                <mesh filename="package://lidar_robot/models/motor.stl" scale="0.001 0.001 0.001"/>
-            </geometry>
-            <material name="aluminium_dark"/>
-        </visual>
-    </link>
-    <joint name="c_clamp_motor_1" type="fixed">
-        <parent link="c_clamp_1"/>
-        <child link="motor_1"/>
-    </joint>
-    <link name="shaft_1">
-        <visual>
-            <origin xyz="${-(c_clamp_dist+0.01)} 0 0.045" rpy="0 0 ${pi}"/>
-            <geometry>
-                <mesh filename="package://lidar_robot/models/motor_shaft.stl" scale="0.001 0.001 0.001"/>
-            </geometry>
-            <material name="plastic"/>
-        </visual>
-    </link>
-    <joint name="motor_shaft_1" type="continuous">
-        <parent link="motor_1"/>
-        <child link="shaft_1"/>
-    </joint>
-    <link name="wheel_1">
-        <visual>
-            <origin xyz="${-(c_clamp_dist+0.03)} 0 0.045" rpy="0 0 ${pi/2}"/>
-            <geometry>
-                <mesh filename="package://lidar_robot/models/wheel2.dae"/>
-            </geometry>
-            <material name="wheel">
-                <texture filename="package://lidar_robot/models/wheel_color.png"/>
-            </material>
-        </visual>
-    </link>
-    <joint name="shaft_wheel_1" type="fixed">
-        <parent link="shaft_1"/>
-        <child link="wheel_1"/>
-    </joint>
-    <!-- =======================================================Wheel 2====================================================================== -->
-    <link name="c_clamp_2">
-        <visual>
-            <origin xyz="0.05 ${c_clamp_dist} 0.09" rpy="${pi/2} 0 -${pi/2}"/>
-            <geometry>
-                <mesh filename="package://lidar_robot/models/c_clamp.stl" scale="0.001 0.001 0.001"/>
-            </geometry>
-            <material name="aluminium"/>
-        </visual>
-    </link>
-    <joint name="base_c_clamp_2" type="fixed">
-        <parent link="base_link"/>
-        <child link="c_clamp_2"/>
-    </joint>
-    <link name="motor_2">
-        <visual>
-            <origin xyz="0 ${(c_clamp_dist-0.012)} 0.045" rpy="${pi/2} -${pi} 0"/>
-            <geometry>
-                <mesh filename="package://lidar_robot/models/motor.stl" scale="0.001 0.001 0.001"/>
-            </geometry>
-            <material name="aluminium_dark"/>
-        </visual>
-    </link>
-    <joint name="c_clamp_motor_2" type="fixed">
-        <parent link="c_clamp_2"/>
-        <child link="motor_2"/>
-    </joint>
-    <link name="shaft_2">
-        <visual>
-            <origin xyz="0 ${(c_clamp_dist+0.01)} 0.045" rpy="0 0 ${pi/2}"/>
-            <geometry>
-                <mesh filename="package://lidar_robot/models/motor_shaft.stl" scale="0.001 0.001 0.001"/>
-            </geometry>
-            <material name="plastic"/>
-        </visual>
-    </link>
-    <joint name="motor_shaft_2" type="continuous">
-        <parent link="motor_2"/>
-        <child link="shaft_2"/>
-    </joint>
-    <link name="wheel_2">
-        <visual>
-            <origin xyz="0 ${(c_clamp_dist+0.03)} 0.045" rpy="0 0 ${pi}"/>
-            <geometry>
-                <mesh filename="package://lidar_robot/models/wheel2.dae"/>
-            </geometry>
-            <material name="wheel">
-                <texture filename="package://lidar_robot/models/wheel_color.png"/>
-            </material>
-        </visual>
-    </link>
-    <joint name="shaft_wheel_2" type="fixed">
-        <parent link="shaft_2"/>
-        <child link="wheel_2"/>
-    </joint>
-    <!-- =======================================================Wheel 3====================================================================== -->
-    <link name="c_clamp_3">
-        <visual>
-            <origin xyz="${c_clamp_dist} -0.05 0.09" rpy="${pi/2} 0 ${pi}"/>
-            <geometry>
-                <mesh filename="package://lidar_robot/models/c_clamp.stl" scale="0.001 0.001 0.001"/>
-            </geometry>
-            <material name="aluminium"/>
-        </visual>
-    </link>
-    <joint name="base_c_clamp_3" type="fixed">
-        <parent link="base_link"/>
-        <child link="c_clamp_3"/>
-    </joint>
-    <link name="motor_3">
-        <visual>
-            <origin xyz="${(c_clamp_dist-0.012)} 0 0.045" rpy="${pi/2} 0 -${pi/2}"/>
-            <geometry>
-                <mesh filename="package://lidar_robot/models/motor.stl" scale="0.001 0.001 0.001"/>
-            </geometry>
-            <material name="aluminium_dark"/>
-        </visual>
-    </link>
-    <joint name="c_clamp_motor_3" type="fixed">
-        <parent link="c_clamp_3"/>
-        <child link="motor_3"/>
-    </joint>
-    <link name="shaft_3">
-        <visual>
-            <origin xyz="${(c_clamp_dist+0.01)} 0 0.045" rpy="0 0 0"/>
-            <geometry>
-                <mesh filename="package://lidar_robot/models/motor_shaft.stl" scale="0.001 0.001 0.001"/>
-            </geometry>
-            <material name="plastic"/>
-        </visual>
-    </link>
-    <joint name="motor_shaft_3" type="continuous">
-        <parent link="motor_3"/>
-        <child link="shaft_3"/>
-    </joint>
-    <link name="wheel_3">
-        <visual>
-            <origin xyz="${(c_clamp_dist+0.03)} 0 0.045" rpy="0 0 ${pi/2}"/>
-            <geometry>
-                <mesh filename="package://lidar_robot/models/wheel2.dae"/>
-            </geometry>
-            <material name="wheel">
-                <texture filename="package://lidar_robot/models/wheel_color.png"/>
-            </material>
-        </visual>
-    </link>
-    <joint name="shaft_wheel_3" type="fixed">
-        <parent link="shaft_3"/>
-        <child link="wheel_3"/>
-    </joint>
-    <!-- =======================================================Wheel 4====================================================================== -->
-    <link name="c_clamp_4">
-        <visual>
-            <origin xyz="-0.05 ${-c_clamp_dist} 0.09" rpy="${pi/2} 0 ${pi/2}"/>
-            <geometry>
-                <mesh filename="package://lidar_robot/models/c_clamp.stl" scale="0.001 0.001 0.001"/>
-            </geometry>
-            <material name="aluminium"/>
-        </visual>
-    </link>
-    <joint name="base_c_clamp_4" type="fixed">
-        <parent link="base_link"/>
-        <child link="c_clamp_4"/>
-    </joint>
-    <link name="motor_4">
-        <visual>
-            <origin xyz="0 ${-(c_clamp_dist-0.012)} 0.045" rpy="${pi/2} 0 ${pi}"/>
-            <geometry>
-                <mesh filename="package://lidar_robot/models/motor.stl" scale="0.001 0.001 0.001"/>
-            </geometry>
-            <material name="aluminium_dark"/>
-        </visual>
-    </link>
-    <joint name="c_clamp_motor_4" type="fixed">
-        <parent link="c_clamp_4"/>
-        <child link="motor_4"/>
-    </joint>
-    <link name="shaft_4">
-        <visual>
-            <origin xyz="0 ${-(c_clamp_dist+0.01)} 0.045" rpy="0 0 ${-pi/2}"/>
-            <geometry>
-                <mesh filename="package://lidar_robot/models/motor_shaft.stl" scale="0.001 0.001 0.001"/>
-            </geometry>
-            <material name="plastic"/>
-        </visual>
-    </link>
-    <joint name="motor_shaft_4" type="continuous">
-        <parent link="motor_4"/>
-        <child link="shaft_4"/>
-    </joint>
-    <link name="wheel_4">
-        <visual>
-            <origin xyz="0 ${-(c_clamp_dist+0.03)} 0.045" rpy="0 0 0"/>
-            <geometry>
-                <mesh filename="package://lidar_robot/models/wheel2.dae"/>
-            </geometry>
-            <material name="wheel">
-                <texture filename="package://lidar_robot/models/wheel_color.png"/>
-            </material>
-        </visual>
-    </link>
-    <joint name="shaft_wheel_4" type="fixed">
-        <parent link="shaft_4"/>
-        <child link="wheel_4"/>
-    </joint>
-    <!-- ======================================================= Top Plate ====================================================================== -->
-    <link name="top_plate">
-        <visual>
-            <origin xyz="0.01 0 0.0836" rpy="${pi/2} 0 0"/>
-            <geometry>
-                <mesh filename="package://lidar_robot/models/top_plate.stl" scale="0.001 0.001 0.001"/>
-            </geometry>
-            <material name="blue"/>
-        </visual>
-    </link>
-    <joint name="base_link_top_plate" type="fixed">
-        <parent link="base_link"/>
-        <child link="top_plate"/>
-    </joint>
-    <!-- ======================================================= Circuit Plate ====================================================================== -->
-    <link name="circuit_plate">
-        <visual>
-            <origin xyz="0 0 0.093" rpy="${pi/2} 0 ${pi/4}"/>
-            <geometry>
-                <mesh filename="package://lidar_robot/models/circuit_plate.stl" scale="0.001 0.001 0.001"/>
-            </geometry>
-            <material name="plastic"/>
-        </visual>
-    </link>
-    <joint name="base_link_circuit_plate" type="fixed">
-        <parent link="top_plate"/>
-        <child link="circuit_plate"/>
-    </joint>
-    <!-- ======================================================= feedback ====================================================================== -->
-    <link name="feedback">
-        <visual>
-            <origin xyz="0.063 0.1 -0.06" rpy="${pi/2} 0 ${pi/4}"/>
-            <geometry>
-                <mesh filename="package://lidar_robot/models/feedback.stl" scale="0.001 0.001 0.001"/>
-            </geometry>
-            <material name="aluminium_dark"/>
-        </visual>
-    </link>
-    <joint name="base_link_feedback" type="fixed">
-        <parent link="base_link"/>
-        <child link="feedback"/>
-    </joint>
     <xacro:macro name="stud" params="myname x y z parent">
         <link name="${myname}">
@@ -306,4 +35,276 @@
         </joint>
     </xacro:macro>
+    <!-- ======================================================= Base Link ====================================================================== -->
+    <link name="base_link">
+        <visual>
+            <origin xyz="0.01 0 0" rpy="${pi/2} 0 0"/>
+            <geometry>
+                <mesh filename="package://lidar_robot/models/base.stl" scale="0.001 0.001 0.001"/>
+            </geometry>
+            <material name="transparent_acrylic"/>
+        </visual>
+    </link>
+    <!-- =======================================================Wheel 1====================================================================== -->
+    <link name="c_clamp_1">
+        <visual>
+            <origin xyz="${-c_clamp_dist} 0.05 0.09" rpy="${pi/2} 0 0"/>
+            <geometry>
+                <mesh filename="package://lidar_robot/models/c_clamp.stl" scale="0.001 0.001 0.001"/>
+            </geometry>
+            <material name="aluminium"/>
+        </visual>
+    </link>
+    <joint name="base_c_clamp_1" type="fixed">
+        <parent link="base_link"/>
+        <child link="c_clamp_1"/>
+    </joint>
+    <link name="motor_1">
+        <visual>
+            <origin xyz="${-(c_clamp_dist-0.012)} 0 0.045" rpy="${pi/2} 0 ${pi/2}"/>
+            <geometry>
+                <mesh filename="package://lidar_robot/models/motor.stl" scale="0.001 0.001 0.001"/>
+            </geometry>
+            <material name="aluminium_dark"/>
+        </visual>
+    </link>
+    <joint name="c_clamp_motor_1" type="fixed">
+        <parent link="c_clamp_1"/>
+        <child link="motor_1"/>
+    </joint>
+    <link name="shaft_1">
+        <visual>
+            <origin xyz="${-(c_clamp_dist+0.01)} 0 0.045" rpy="0 0 ${pi}"/>
+            <geometry>
+                <mesh filename="package://lidar_robot/models/motor_shaft.stl" scale="0.001 0.001 0.001"/>
+            </geometry>
+            <material name="plastic"/>
+        </visual>
+    </link>
+    <joint name="motor_shaft_1" type="continuous">
+        <parent link="motor_1"/>
+        <child link="shaft_1"/>
+    </joint>
+    <link name="wheel_1">
+        <visual>
+            <origin xyz="${-(c_clamp_dist+0.03)} 0 0.045" rpy="0 0 ${pi/2}"/>
+            <geometry>
+                <mesh filename="package://lidar_robot/models/wheel2.dae"/>
+            </geometry>
+            <material name="wheel">
+                <texture filename="package://lidar_robot/models/wheel_color.png"/>
+            </material>
+        </visual>
+    </link>
+    <joint name="shaft_wheel_1" type="fixed">
+        <parent link="shaft_1"/>
+        <child link="wheel_1"/>
+    </joint>
+    <!-- =======================================================Wheel 2====================================================================== -->
+    <link name="c_clamp_2">
+        <visual>
+            <origin xyz="0.05 ${c_clamp_dist} 0.09" rpy="${pi/2} 0 -${pi/2}"/>
+            <geometry>
+                <mesh filename="package://lidar_robot/models/c_clamp.stl" scale="0.001 0.001 0.001"/>
+            </geometry>
+            <material name="aluminium"/>
+        </visual>
+    </link>
+    <joint name="base_c_clamp_2" type="fixed">
+        <parent link="base_link"/>
+        <child link="c_clamp_2"/>
+    </joint>
+    <link name="motor_2">
+        <visual>
+            <origin xyz="0 ${(c_clamp_dist-0.012)} 0.045" rpy="${pi/2} -${pi} 0"/>
+            <geometry>
+                <mesh filename="package://lidar_robot/models/motor.stl" scale="0.001 0.001 0.001"/>
+            </geometry>
+            <material name="aluminium_dark"/>
+        </visual>
+    </link>
+    <joint name="c_clamp_motor_2" type="fixed">
+        <parent link="c_clamp_2"/>
+        <child link="motor_2"/>
+    </joint>
+    <link name="shaft_2">
+        <visual>
+            <origin xyz="0 ${(c_clamp_dist+0.01)} 0.045" rpy="0 0 ${pi/2}"/>
+            <geometry>
+                <mesh filename="package://lidar_robot/models/motor_shaft.stl" scale="0.001 0.001 0.001"/>
+            </geometry>
+            <material name="plastic"/>
+        </visual>
+    </link>
+    <joint name="motor_shaft_2" type="continuous">
+        <parent link="motor_2"/>
+        <child link="shaft_2"/>
+    </joint>
+    <link name="wheel_2">
+        <visual>
+            <origin xyz="0 ${(c_clamp_dist+0.03)} 0.045" rpy="0 0 ${pi}"/>
+            <geometry>
+                <mesh filename="package://lidar_robot/models/wheel2.dae"/>
+            </geometry>
+            <material name="wheel">
+                <texture filename="package://lidar_robot/models/wheel_color.png"/>
+            </material>
+        </visual>
+    </link>
+    <joint name="shaft_wheel_2" type="fixed">
+        <parent link="shaft_2"/>
+        <child link="wheel_2"/>
+    </joint>
+    <!-- =======================================================Wheel 3====================================================================== -->
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
Commit message: Added RPlidar Bottom

File: src/lidar_robot/xacro/robot.xacro (robot description, xacro)
@@ -3,4 +3,7 @@
     <material name="transparent_acrylic">
         <color rgba="0.8 0.8 0.8 0.4"/>
+    </material>
+    <material name="transparent_acrylic_dark">
+        <color rgba="0.4 0.4 0.4 0.4"/>
     </material>
     <material name="aluminium">
@@ -322,5 +325,5 @@
                 <mesh filename="package://lidar_robot/models/lidar_base.stl" scale="0.001 0.001 0.001"/>
             </geometry>
-            <material name="transparent_acrylic"/>
+            <material name="transparent_acrylic_dark"/>
         </visual>
     </link>
@@ -333,3 +336,17 @@
     <xacro:stud myname="s11" x="-0.0321" y="-0.041" z="0.098" parent="circuit_plate"/>
     <xacro:stud myname="s12" x="-0.0321" y="0.021" z="0.098" parent="circuit_plate"/>
+    <!-- ======================================================= RPlidar ====================================================================== -->
+    <link name="lidar_bottom">
+        <visual>
+            <origin xyz="0.0 0 0.161" rpy="${pi/2} 0 ${-pi/2}"/>
+            <geometry>
+                <mesh filename="package://lidar_robot/models/lidar_bottom.stl" scale="0.001 0.001 0.001"/>
+            </geometry>
+            <material name="aluminium"/>
+        </visual>
+    </link>
+    <joint name="lidar_base_lidar_bottom" type="fixed">
+        <parent link="lidar_base"/>
+        <child link="lidar_bottom"/>
+    </joint>
 </robot>

Commit message: Added Lidar UP updated stud.stl with proper binary encoding

File: src/lidar_robot/xacro/robot.xacro (robot description, xacro)
@@ -15,4 +15,7 @@
     <material name="plastic">
         <color rgba="0.95 0.95 0.95 1"/>
+    </material>
+    <material name="black_plastic">
+        <color rgba="0.0 0.0 0.0 1"/>
     </material>
     <material name="blue">
@@ -350,3 +353,16 @@
         <child link="lidar_bottom"/>
     </joint>
+    <link name="lidar_up">
+        <visual>
+            <origin xyz="0.0 0 0.158" rpy="${pi/2} 0 ${-pi/2}"/>
+            <geometry>
+                <mesh filename="package://lidar_robot/models/lidar_up.stl" scale="0.001 0.001 0.001"/>
+            </geometry>
+            <material name="black_plastic"/>
+        </visual>
+    </link>
+    <joint name="lidar_bottom_lidar_up" type="fixed">
+        <parent link="lidar_bottom"/>
+        <child link="lidar_up"/>
+    </joint>
 </robot>

Commit message: Added Gazebo

File: src/lidar_robot/xacro/robot.xacro (robot description, xacro)
@@ -50,4 +50,13 @@
             <material name="transparent_acrylic"/>
         </visual>
+        <inertial>
+            <mass value="8"/>
+            <inertia ixx="0.000231" ixy="0.0" ixz="0.0" iyy="0.000439" iyz="-0.000001" izz="0.999454"/>
+        </inertial>
+        <collision>
+            <geometry>
+                <box size="0.613 0.613 0.21"/>
+            </geometry>
+        </collision>
     </link>
     <!-- =======================================================Wheel 1====================================================================== -->

Commit message: Updated URDF with Gazebo wheels

File: src/lidar_robot/xacro/robot.xacro (robot description, xacro)
@@ -41,4 +41,22 @@
         </joint>
     </xacro:macro>
+    <xacro:macro name="wheel">
+        <visual>
+            <origin xyz="0.02 0 0" rpy="0 0 ${pi/2}"/>
+            <geometry>
+                <mesh filename="package://lidar_robot/models/wheel2.dae"/>
+            </geometry>
+        </visual>
+        <inertial>
+            <mass value="0.5"/>
+            <inertia ixx="0.0" ixy="0.0" ixz="0.0" iyy="0.000001" iyz="0.0" izz="0.0"/>
+        </inertial>
+        <collision>
+            <origin xyz="0.027 0 0.0" rpy="0 ${pi/2} 0"/>
+            <geometry>
+                <cylinder length="0.045" radius="0.08"/>
+            </geometry>
+        </collision>
+    </xacro:macro>
     <!-- ======================================================= Base Link ====================================================================== -->
     <link name="base_link">
@@ -55,6 +73,13 @@
         </inertial>
         <collision>
-            <geometry>
-                <box size="0.613 0.613 0.21"/>
+            <origin xyz="0 0 0.05" rpy="0 0 ${pi/4}"/>
+            <geometry>
+                <box size="0.52 0.52 0.11"/>
+            </geometry>
+        </collision>
+        <collision>
+            <origin xyz="0 0 0.07" rpy="0 0 0"/>
+            <geometry>
+                <cylinder length="0.205" radius=".07"/>
             </geometry>
         </collision>
@@ -97,5 +122,5 @@
     </link>
     <joint name="motor_shaft_1" type="continuous">
-        <parent link="motor_1"/>
+        <parent link="base_link"/>
         <child link="shaft_1"/>
         <axis xyz="1 0 0"/>
@@ -103,10 +128,5 @@
     </joint>
     <link name="wheel_1">
-        <visual>
-            <origin xyz="0.02 0 0" rpy="0 0 ${pi/2}"/>
-            <geometry>
-                <mesh filename="package://lidar_robot/models/wheel2.dae"/>
-            </geometry>
-        </visual>
+        <xacro:wheel/>
     </link>
     <joint name="shaft_wheel_1" type="fixed">
@@ -151,15 +171,10 @@
     </link>
     <joint name="motor_shaft_2" type="continuous">
-        <parent link="motor_2"/>
+        <parent link="base_link"/>
         <child link="shaft_2"/>
         <origin xyz="0 ${(c_clamp_dist+0.01)} 0.045" rpy="0 0 ${pi/2}"/>
     </joint>
     <link name="wheel_2">
-        <visual>
-            <origin xyz="0.02 0 0" rpy="0 0 ${pi/2}"/>
-            <geometry>
-                <mesh filename="package://lidar_robot/models/wheel2.dae"/>
-            </geometry>
-        </visual>
+        <xacro:wheel/>
     </link>
     <joint name="shaft_wheel_2" type="fixed">
@@ -204,15 +219,10 @@
     </link>
     <joint name="motor_shaft_3" type="continuous">
-        <parent link="motor_3"/>
+        <parent link="base_link"/>
         <child link="shaft_3"/>
         <origin xyz="${(c_clamp_dist+0.01)} 0 0.045" rpy="0 0 0"/>
     </joint>
     <link name="wheel_3">
-        <visual>
-            <origin xyz="0.02 0 0" rpy="0 0 ${pi/2}"/>
-            <geometry>
-                <mesh filename="package://lidar_robot/models/wheel2.dae"/>
-            </geometry>
-        </visual>
+        <xacro:wheel/>
     </link>
     <joint name="shaft_wheel_3" type="fixed">
@@ -257,15 +267,10 @@
     </link>
     <joint name="motor_shaft_4" type="continuous">
-        <parent link="motor_4"/>
+        <parent link="base_link"/>
         <child link="shaft_4"/>
         <origin xyz="0 ${-(c_clamp_dist+0.01)} 0.045" rpy="0 0 ${-pi/2}"/>
     </joint>
     <link name="wheel_4">
-        <visual>
-            <origin xyz="0.02 0 0" rpy="0 0 ${pi/2}"/>
-            <geometry>
-                <mesh filename="package://lidar_robot/models/wheel2.dae"/>
-            </geometry>
-        </visual>
+        <xacro:wheel/>
     </link>
     <joint name="shaft_wheel_4" type="fixed">
