Commit message: Gazebo is functioning

File: src/lidar_robot/xacro/robot.xacro (robot description, xacro)
@@ -373,3 +373,51 @@
         <child link="lidar_up"/>
     </joint>
+    <link name="rplidar_frame">
+        <visual>
+            <geometry>
+                <sphere radius="0.001"/>
+            </geometry>
+            <material name="blue"/>
+        </visual>
+    </link>
+    <joint name="base_link_rplidar_frame" type="fixed">
+        <origin xyz="0.0 0 0.16" rpy="0 0 0"/>
+        <parent link="base_link"/>
+        <child link="rplidar_frame"/>
+    </joint>
+    <gazebo reference="rplidar_frame">
+        <sensor type="ray" name="rplidar_sensor">
+            <pose>0 0 0 0 0 0</pose>
+            <visualize>true</visualize>
+            <update_rate>8</update_rate>
+            <ray>
+                <scan>
+                    <horizontal>
+                        <samples>360</samples>
+                        <resolution>1</resolution>
+                        <min_angle>0</min_angle>
+                        <max_angle>${pi*2}</max_angle>
+                    </horizontal>
+                </scan>
+                <range>
+                    <min>0.2</min>
+                    <max>6.0</max>
+                    <resolution>0.5</resolution>
+                </range>
+                <noise>
+                    <type>gaussian</type>
+                    <!-- Noise parameters based on published spec for Hokuyo laser
+               achieving "+-30mm" accuracy at range < 10m.  A mean of 0.0m and
+               stddev of 0.01m will put 99.7% of samples within 0.03m of the true
+               reading. -->
+                    <mean>0.0</mean>
+                    <stddev>0.01</stddev>
+                </noise>
+            </ray>
+            <plugin name="gazebo_ros_rplidar_controller" filename="libgazebo_ros_laser.so">
+                <topicName>/scan</topicName>
+                <frameName>/rplidar_frame</frameName>
+            </plugin>
+        </sensor>
+    </gazebo>
 </robot>

Commit message: Added ROS-Control
Partially added, gazebo model does not place shaft correctly yet.

File: src/lidar_robot/xacro/robot.xacro (robot description, xacro)
@@ -1,28 +1,10 @@
 <?xml version="1.0"?>
 <robot xmlns:xacro="http://www.ros.org/wiki/xacro" name="lidar_robot">
-    <material name="transparent_acrylic">
-        <color rgba="0.8 0.8 0.8 0.4"/>
-    </material>
-    <material name="transparent_acrylic_dark">
-        <color rgba="0.4 0.4 0.4 0.4"/>
-    </material>
-    <material name="aluminium">
-        <color rgba="0.8 0.8 0.8 1"/>
-    </material>
-    <material name="aluminium_dark">
-        <color rgba="0.6 0.6 0.6 1"/>
-    </material>
-    <material name="plastic">
-        <color rgba="0.95 0.95 0.95 1"/>
-    </material>
-    <material name="black_plastic">
-        <color rgba="0.0 0.0 0.0 1"/>
-    </material>
-    <material name="blue">
-        <color rgba="0 0 1.0 1"/>
-    </material>
-    <material name="bronze">
-        <color rgba="0.8039 0.498 0.196 1"/>
-    </material>
+    <xacro:include filename="$(find lidar_robot)/xacro/materials.xacro"/>
+    <gazebo>
+        <plugin name="gazebo_ros_control" filename="libgazebo_ros_control.so">
+            <robotNamespace>/lidar_robot</robotNamespace>
+        </plugin>
+    </gazebo>
     <xacro:property name="c_clamp_dist" value="0.31"/>
     <xacro:macro name="stud" params="myname x y z parent">
@@ -134,4 +116,14 @@
         <child link="wheel_1"/>
     </joint>
+    <transmission name="trans_m1">
+        <type>transmission_interface/SimpleTransmission</type>
+        <joint name="motor_shaft_1">
+            <hardwareInterface>EffortJointInterface</hardwareInterface>
+        </joint>
+        <actuator name="motor1">
+            <hardwareInterface>EffortJointInterface</hardwareInterface>
+            <mechanicalReduction>1</mechanicalReduction>
+        </actuator>
+    </transmission>
     <!-- =======================================================Wheel 2====================================================================== -->
     <link name="c_clamp_2">
@@ -182,4 +174,14 @@
         <child link="wheel_2"/>
     </joint>
+    <transmission name="trans_m2">
+        <type>transmission_interface/SimpleTransmission</type>
+        <joint name="motor_shaft_2">
+            <hardwareInterface>EffortJointInterface</hardwareInterface>
+        </joint>
+        <actuator name="motor2">
+            <hardwareInterface>EffortJointInterface</hardwareInterface>
+            <mechanicalReduction>1</mechanicalReduction>
+        </actuator>
+    </transmission>
     <!-- =======================================================Wheel 3====================================================================== -->
     <link name="c_clamp_3">
@@ -230,4 +232,14 @@
         <child link="wheel_3"/>
     </joint>
+    <transmission name="trans_m3">
+        <type>transmission_interface/SimpleTransmission</type>
+        <joint name="motor_shaft_3">
+            <hardwareInterface>EffortJointInterface</hardwareInterface>
+        </joint>
+        <actuator name="motor3">
+            <hardwareInterface>EffortJointInterface</hardwareInterface>
+            <mechanicalReduction>1</mechanicalReduction>
+        </actuator>
+    </transmission>
     <!-- =======================================================Wheel 4====================================================================== -->
     <link name="c_clamp_4">
@@ -278,4 +290,14 @@
         <child link="wheel_4"/>
     </joint>
+    <transmission name="trans_m4">
+        <type>transmission_interface/SimpleTransmission</type>
+        <joint name="motor_shaft_4">
+            <hardwareInterface>EffortJointInterface</hardwareInterface>
+        </joint>
+        <actuator name="motor4">
+            <hardwareInterface>EffortJointInterface</hardwareInterface>
+            <mechanicalReduction>1</mechanicalReduction>
+        </actuator>
+    </transmission>
     <!-- ======================================================= Top Plate ====================================================================== -->
     <link name="top_plate">

Commit message: Removed Controller setup
Removed controller as the real bot does not have any feedback on wheels, so cannot use the PID control, though gazebo provides it.

File: src/lidar_robot/xacro/robot.xacro (robot description, xacro)
@@ -2,9 +2,4 @@
 <robot xmlns:xacro="http://www.ros.org/wiki/xacro" name="lidar_robot">
     <xacro:include filename="$(find lidar_robot)/xacro/materials.xacro"/>
-    <gazebo>
-        <plugin name="gazebo_ros_control" filename="libgazebo_ros_control.so">
-            <robotNamespace>/lidar_robot</robotNamespace>
-        </plugin>
-    </gazebo>
     <xacro:property name="c_clamp_dist" value="0.31"/>
     <xacro:macro name="stud" params="myname x y z parent">
@@ -116,14 +111,4 @@
         <child link="wheel_1"/>
     </joint>
-    <transmission name="trans_m1">
-        <type>transmission_interface/SimpleTransmission</type>
-        <joint name="motor_shaft_1">
-            <hardwareInterface>EffortJointInterface</hardwareInterface>
-        </joint>
-        <actuator name="motor1">
-            <hardwareInterface>EffortJointInterface</hardwareInterface>
-            <mechanicalReduction>1</mechanicalReduction>
-        </actuator>
-    </transmission>
     <!-- =======================================================Wheel 2====================================================================== -->
     <link name="c_clamp_2">
@@ -174,14 +159,4 @@
         <child link="wheel_2"/>
     </joint>
-    <transmission name="trans_m2">
-        <type>transmission_interface/SimpleTransmission</type>
-        <joint name="motor_shaft_2">
-            <hardwareInterface>EffortJointInterface</hardwareInterface>
-        </joint>
-        <actuator name="motor2">
-            <hardwareInterface>EffortJointInterface</hardwareInterface>
-            <mechanicalReduction>1</mechanicalReduction>
-        </actuator>
-    </transmission>
     <!-- =======================================================Wheel 3====================================================================== -->
     <link name="c_clamp_3">
@@ -232,14 +207,4 @@
         <child link="wheel_3"/>
     </joint>
-    <transmission name="trans_m3">
-        <type>transmission_interface/SimpleTransmission</type>
-        <joint name="motor_shaft_3">
-            <hardwareInterface>EffortJointInterface</hardwareInterface>
-        </joint>
-        <actuator name="motor3">
-            <hardwareInterface>EffortJointInterface</hardwareInterface>
-            <mechanicalReduction>1</mechanicalReduction>
-        </actuator>
-    </transmission>
     <!-- =======================================================Wheel 4====================================================================== -->
     <link name="c_clamp_4">
@@ -290,14 +255,4 @@
         <child link="wheel_4"/>
     </joint>
-    <transmission name="trans_m4">
-        <type>transmission_interface/SimpleTransmission</type>
-        <joint name="motor_shaft_4">
-            <hardwareInterface>EffortJointInterface</hardwareInterface>
-        </joint>
-        <actuator name="motor4">
-            <hardwareInterface>EffortJointInterface</hardwareInterface>
-            <mechanicalReduction>1</mechanicalReduction>
-        </actuator>
-    </transmission>
     <!-- ======================================================= Top Plate ====================================================================== -->
     <link name="top_plate">

Commit message: Updated xacro with proper frames

File: src/lidar_robot/xacro/robot.xacro (robot description, xacro)
@@ -281,5 +281,5 @@
     <link name="circuit_plate">
         <visual>
-            <origin xyz="0 0 0.093" rpy="${pi/2} 0 ${pi/4}"/>
+            <origin xyz="0 0 0.093" rpy="${pi/2} 0 ${-5*pi/4}"/>
             <geometry>
                 <mesh filename="package://lidar_robot/models/circuit_plate.stl" scale="0.001 0.001 0.001"/>
@@ -317,5 +317,5 @@
     <link name="lidar_base">
         <visual>
-            <origin xyz="0.0 -0.01 0.1134" rpy="${pi/2} 0 ${-pi/2}"/>
+            <origin xyz="0.01 0 0.1134" rpy="${pi/2} 0 0"/>
             <geometry>
                 <mesh filename="package://lidar_robot/models/lidar_base.stl" scale="0.001 0.001 0.001"/>
@@ -328,12 +328,12 @@
         <child link="lidar_base"/>
     </joint>
-    <xacro:stud myname="s9" x="0.0321" y="0.021" z="0.098" parent="circuit_plate"/>
-    <xacro:stud myname="s10" x="0.0321" y="-0.041" z="0.098" parent="circuit_plate"/>
-    <xacro:stud myname="s11" x="-0.0321" y="-0.041" z="0.098" parent="circuit_plate"/>
-    <xacro:stud myname="s12" x="-0.0321" y="0.021" z="0.098" parent="circuit_plate"/>
+    <xacro:stud myname="s9" x="-0.021" y="0.0321" z="0.098" parent="lidar_base"/>
+    <xacro:stud myname="s10" x="0.041" y="0.0321" z="0.098" parent="lidar_base"/>
+    <xacro:stud myname="s11" x="0.041" y="-0.0321" z="0.098" parent="lidar_base"/>
+    <xacro:stud myname="s12" x="-0.021" y="-0.0321" z="0.098" parent="lidar_base"/>
     <!-- ======================================================= RPlidar ====================================================================== -->
     <link name="lidar_bottom">
         <visual>
-            <origin xyz="0.0 0 0.161" rpy="${pi/2} 0 ${-pi/2}"/>
+            <origin xyz="0.0 0 0.161" rpy="${pi/2} 0 0"/>
             <geometry>
                 <mesh filename="package://lidar_robot/models/lidar_bottom.stl" scale="0.001 0.001 0.001"/>
@@ -348,5 +348,5 @@
     <link name="lidar_up">
         <visual>
-            <origin xyz="0.0 0 0.158" rpy="${pi/2} 0 ${-pi/2}"/>
+            <origin xyz="0.0 0 0.158" rpy="${pi/2} 0 0"/>
             <geometry>
                 <mesh filename="package://lidar_robot/models/lidar_up.stl" scale="0.001 0.001 0.001"/>
@@ -407,3 +407,42 @@
         </sensor>
     </gazebo>
+    <link name="x">
+        <visual>
+            <origin xyz="1.0 0 0" rpy="0 0 0"/>
+            <geometry>
+                <sphere radius="0.1"/>
+            </geometry>
+            <material name="blue"/>
+        </visual>
+    </link>
+    <joint name="base_link_x" type="fixed">
+        <parent link="base_link"/>
+        <child link="x"/>
+    </joint>
+    <link name="y">
+        <visual>
+            <origin xyz="0 1 0" rpy="0 0 0"/>
+            <geometry>
+                <sphere radius="0.1"/>
+            </geometry>
+            <material name="bronze"/>
+        </visual>
+    </link>
+    <joint name="base_link_y" type="fixed">
+        <parent link="base_link"/>
+        <child link="y"/>
+    </joint>
+    <link name="imu">
+        <visual>
+            <origin xyz="0.16 0.05 0.02" rpy="0 0 0"/>
+            <geometry>
+                <box size="0.05 0.03 0.004"/>
+            </geometry>
+            <material name="blue"/>
+        </visual>
+    </link>
+    <joint name="base_link_imu" type="fixed">
+        <parent link="base_link"/>
+        <child link="imu"/>
+    </joint>
 </robot>
